Commit message: robot is now in the right shape (probobly)

File: RL_robot/model/robot.xacro (robot description, xacro)
@@ -10,13 +10,13 @@
 <xacro:property name="PI" value="3.14159265359"/>
 <!-- Body Dimensions -->
-<!-- R = radius of robot -->
-<!-- H = height of robot -->
-<xacro:property name="R" value="0.25"/>
-<xacro:property name="H" value="0.35"/>
+<!-- R = side of robot body -->
+<!-- H = height of robot body -->
+<xacro:property name="R" value="0.3"/>
+<xacro:property name="H" value="0.25"/>
 <!-- Wheels Dimensions -->
 <!-- r = wheels && caster radius -->
 <!-- w = wheels width -->
-<xacro:property name="r" value="0.1"/>
-<xacro:property name="w" value="0.04"/>
+<xacro:property name="r" value="0.034"/>
+<xacro:property name="w" value="0.028"/>
 <!-- Lengths to centers -->
 <!-- s1 = length from c1 to c2 -->
@@ -24,6 +24,6 @@
 <!-- s3 = length from c2 to c5 -->
 <xacro:property name="s1" value="${H/2+r}"/>
-<xacro:property name="s2" value="${R}"/>
-<xacro:property name="s3" value="${s2/2.0}"/>
+<xacro:property name="s2" value="${R/2.0}"/>
+<xacro:property name="s3" value="${R/2.0-0.03}"/>
 <!-- ##################################################### -->
 <!--                    Mass && Inertia                    -->
@@ -58,5 +58,5 @@
 <!-- MASSES -->
 <!-- Body -->
-<xacro:property name="m1" value="${d1*PI*H*R*R}"/>
+<xacro:property name="m1" value="${d1*H*R*R}"/>
 <!-- Wheel -->
 <xacro:property name="m2" value="${d2*PI*w*r*r}"/>
@@ -64,6 +64,7 @@
 <xacro:property name="m3" value="${d3*(4.0/3.0)*PI*r*r*r}"/>
 <!-- Momments of inertia Body -->
-<xacro:property name="I_body" value="${(1.0/12.0)*m1*(3.0*R*R+H*H)}"/>
-<xacro:property name="Iz_body" value="${0.5*m1*R*R}"/>
+<xacro:property name="Ix_body" value="${(1.0/12.0)*m1*(R*R+H*H)}"/>
+<xacro:property name="Iy_body" value="${(1.0/12.0)*m1*(R*R+H*H)}"/>
+<xacro:property name="Iz_body" value="${(1.0/12.0)*m1*(R*R+R*R)}"/>
 <!-- Momments of inertia Wheel -->
 <xacro:property name="I_wheel" value="${(1.0/12.0)*m2*(3.0*r*r+w*w)}"/>
@@ -76,5 +77,5 @@
     <origin rpy="0 0 0" xyz="0 0 ${s1}"/>
     <mass value="${m1}"/>
-    <inertia ixx="${I_body}" ixy="0.0" ixz="0.0" iyy="${I_body}" iyz="0.0" izz="${Iz_body}"/>
+    <inertia ixx="${Ix_body}" ixy="0.0" ixz="0.0" iyy="${Iy_body}" iyz="0.0" izz="${Iz_body}"/>
     </inertial>
 </xacro:macro>
@@ -112,5 +113,5 @@
     <visual>
         <geometry>
-            <cylinder length="${H}" radius="${R}"/>
+            <box size="${R} ${R} ${H}"/>
         </geometry>
         <origin rpy="0 0 0" xyz="0 0 ${s1}"/>
@@ -118,5 +119,5 @@
     <collision>
         <geometry>
-            <cylinder length="${H}" radius="${R}"/>
+            <box size="${R} ${R} ${H}"/>
         </geometry>
         <origin rpy="0 0 0" xyz="0 0 ${s1}"/>
@@ -129,5 +130,5 @@
     <parent link="body_link"/>
     <child link="wheel1_link"/>
-    <origin rpy="0 0 0" xyz="0 ${-s2} ${r}"/>
+    <origin rpy="0 0 0" xyz="${-s3} ${-s2} ${r}"/>
     <axis xyz="0 1 0"/>
     <limit effort="50000" velocity="10"/>
@@ -154,5 +155,5 @@
     <parent link="body_link"/>
     <child link="wheel2_link"/>
-    <origin rpy="0 0 0" xyz="0 ${s2} ${r}"/>
+    <origin rpy="0 0 0" xyz="${-s3} ${s2} ${r}"/>
     <axis xyz="0 1 0"/>
     <limit effort="50000" velocity="10"/>
@@ -187,11 +188,11 @@
             <sphere radius="${r}"/>
         </geometry>
-        <origin rpy="0 0 0" xyz="${s3} 0 ${r}"/>
-    </visual>
-    <collision>
-        <geometry>
-            <sphere radius="${r}"/>
-        </geometry>
-        <origin rpy="0 0 0" xyz="${s3} 0 ${r}"/>
+        <origin rpy="0 0 0" xyz="${s3} ${s3} ${r}"/>
+    </visual>
+    <collision>
+        <geometry>
+            <sphere radius="${r}"/>
+        </geometry>
+        <origin rpy="0 0 0" xyz="${s3} ${s3} ${r}"/>
     </collision>
     <xacro:inertia_caster />
@@ -208,11 +209,11 @@
             <sphere radius="${r}"/>
         </geometry>
-        <origin rpy="0 0 0" xyz="${-s3} 0 ${r}"/>
-    </visual>
-    <collision>
-        <geometry>
-            <sphere radius="${r}"/>
-        </geometry>
-        <origin rpy="0 0 0" xyz="${-s3} 0 ${r}"/>
+        <origin rpy="0 0 0" xyz="${s3} ${-s3} ${r}"/>
+    </visual>
+    <collision>
+        <geometry>
+            <sphere radius="${r}"/>
+        </geometry>
+        <origin rpy="0 0 0" xyz="${s3} ${-s3} ${r}"/>
     </collision>
     <xacro:inertia_caster />
@@ -229,5 +230,5 @@
             <cylinder length="${2*w}" radius="${r}"/>
         </geometry>
-        <origin rpy="0 0 0" xyz="0 0 ${(H/2)+w+s1}"/>
+        <origin rpy="0 0 0" xyz="${-s3} 0 ${(H/2)+w+s1}"/>
     </visual>
     <collision>
@@ -235,5 +236,5 @@
             <cylinder length="${2*w}" radius="${r}"/>
         </geometry>
-        <origin rpy="0 0 0" xyz="0 0 ${(H/2)+w+s1}"/>
+        <origin rpy="0 0 0" xyz="${-s3} 0 ${(H/2)+w+s1}"/>
     </collision>
     <xacro:inertia_wheel />

Commit message: fixed asymmetric acceleration deceleration, improved reward func, need to fix reward buffer

File: RL_robot/model/robot.xacro (robot description, xacro)
@@ -31,9 +31,9 @@
 <!-- Material density -->
 <!-- Body material density -->
-<xacro:property name="d1" value="2710.0"/>
+<xacro:property name="d1" value="155.0"/>
 <!-- Wheel material density -->
-<xacro:property name="d2" value="2710.0"/>
+<xacro:property name="d2" value="100.0"/>
 <!-- Caster material density -->
-<xacro:property name="d3" value="2710.0"/>
+<xacro:property name="d3" value="130.0"/>
 <!-- ################### MASS, VOLUME, CENTER OF MASS EQU ################### -->
 <!-- Volumes -->
@@ -132,6 +132,6 @@
     <origin rpy="0 0 0" xyz="${-s3} ${-s2} ${r}"/>
     <axis xyz="0 1 0"/>
-    <limit effort="50000" velocity="10"/>
-    <dynamics damping="1.0" friction="1.0"/>
+    <limit effort="0.7" velocity="30.0"/>
+    <dynamics damping="0.05" friction="0.05"/>
 </joint>
 <!-- wheel1 link -->
@@ -157,6 +157,6 @@
     <origin rpy="0 0 0" xyz="${-s3} ${s2} ${r}"/>
     <axis xyz="0 1 0"/>
-    <limit effort="50000" velocity="10"/>
-    <dynamics damping="1.0" friction="1.0"/>
+    <limit effort="0.7" velocity="30.0"/>
+    <dynamics damping="0.05" friction="0.05"/>
 </joint>
 <!-- wheel2 link -->

Commit message: added more worlds

File: RL_robot/model/robot.xacro (robot description, xacro)
@@ -17,5 +17,5 @@
 <!-- r = wheels && caster radius -->
 <!-- w = wheels width -->
-<xacro:property name="r" value="0.034"/>
+<xacro:property name="r" value="0.08"/>
 <xacro:property name="w" value="0.028"/>
 <!-- Lengths to centers -->

Commit message: fixed weird speeds

File: RL_robot/model/robot.xacro (robot description, xacro)
@@ -17,5 +17,5 @@
 <!-- r = wheels && caster radius -->
 <!-- w = wheels width -->
-<xacro:property name="r" value="0.08"/>
+<xacro:property name="r" value="0.034"/>  <!-- irl it's 0.034 -->
 <xacro:property name="w" value="0.028"/>
 <!-- Lengths to centers -->
